File: Eagle/WaterLevelDisplay/WaterLevelDisplay_v1-0.brd (EAGLE design)
At the start: 88.9 x 99.1 mm, 23 parts, among them J12 POWER_JACKPTH_BREAD, J7 RJ45

Commit message: first round of layout
Parts:
- removed C2: 0.01uF, SparkFun-Passives:CAP-PTH-5MM
- removed J10: (no value), SparkFun-Connectors:1X02
- removed LED1: (no value), adafruit:LED5MM
- removed R10: 330, resistor:0204/5
- added CN1: (no value), adafruit:JST-PH-2-SMT-RA
- added J5: (no value), SparkFun-Connectors:1X20_NOSILK
- added OK1: SFH620A, optocoupler:DIL04
- R5: value 22K -> 5K
- R6: value 10K -> 8K
- moved R5 41.8 mm to (66.0, 25.4)
- moved R6 34.7 mm to (69.8, 25.4), turned to 270 degrees
Connections:
- removed net MOTION: J7.4
- removed net N$6: C2.1, R5.1, R6.2
- removed net PHOTOCELL: J7.5
- new net CURTRANS_A: J7.4, OK1.2
- new net CURTRANS_B: J7.5, OK1.1
- new net N$10: J2.8, J5.8
- new net N$11: J2.9, J5.9
- new net N$12: J2.10, J5.10
- new net N$13: J2.11, J5.11
- new net N$14: J2.12, J5.12
- new net N$16: J2.13, J5.13
- new net N$19: J2.14, J5.14
- new net N$2: J2.2, J5.2
- new net N$20: J2.15, J5.15
- new net N$21: J2.16, J5.16
- new net N$22: J2.17, J5.17
- new net N$23: J2.18, J5.18
- new net N$24: J2.19, J5.19
- new net N$25: J2.20, J5.20
- new net N$27: J1.8, J4.7
- new net N$28: J1.19, J3.12
- new net N$29: J1.20, J3.11
- new net N$3: J2.3, J5.3
- new net N$30: J1.10, J4.6
- new net N$31: J3.9, OK1.4
- new net N$32: J1.7, J4.8
- new net N$33: J1.9, J3.7
- new net N$4: J2.4, J5.4
- new net N$5: J2.5, J5.5
- new net N$7: J2.6, J5.6
- new net N$8: J2.7, J5.7
- net GND: now also CN1.2, J1.1, J1.15, J12.GND, J2.1, J3.13, J5.1, OK1.3; no longer C2.2, J10.2, J12.PWR, LED1.K, S1.3
- net MISO: now also J1.5, J3.4
- net MOSI: now also J1.6, J3.5
- net N$1: now also CN1.1, S1.3; no longer LED1.A, R10.2
- net N$15: now also J3.1, J3.8; no longer R10.1
- net N$17: now also J12.PWR, J4.10, R5.2; no longer J10.1, J12.GND
- net N$18: now also J3.10, R5.1, R6.2; no longer R5.2
- net N$9: now also J4.12
- net RST: now also J3.16
- net SCK: now also J1.4, J3.6
- net VCC: now also J1.2, J3.15
Routing:
- net MISO: track 0.00 -> 108.9 mm
- net MOSI: track 0.00 -> 100.3 mm
- net VCC: track 0.00 -> 95.1 mm
- net RST: track 0.00 -> 90.2 mm
- net SCK: track 0.00 -> 88.7 mm
- net N$28: track 0.00 -> 66.9 mm
- net N$29: track 0.00 -> 66.9 mm
- net N$31: track 0.00 -> 49.6 mm
- net N$27: track 0.00 -> 43.5 mm
- net N$32: track 0.00 -> 43.5 mm
- net N$30: track 0.00 -> 42.4 mm
- net N$17: track 0.00 -> 38.8 mm
- net N$33: track 0.00 -> 32.2 mm
- net N$15: track 0.00 -> 21.4 mm
- net N$9: track 0.00 -> 19.4 mm
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- added copper zone on layer 1, net GND
- added copper zone on layer 16, net GND
Other:
- board text removed: "+"
- board text removed: "Shdn in gnd out"

Commit message: Add files via upload
Parts:
- added C1, C2: 330uF, SparkFun-Capacitors:CPOL-RADIAL-100UF-25V
- added D1: 6V Zener, SparkFun-DiscreteSemi:DIODE-ZENER
- added J10: (no value), SparkFun-Connectors:1X02
- added J6, J8, J9: (no value), SparkFun-Connectors:1X04
- moved R5 0.64 mm to (65.4, 25.4)
- moved U$2 0.64 mm to (84.5, 34.3)
- moved U$4 0.64 mm to (84.5, 16.5)
- moved J3 0.63 mm to (42.5, 15.2)
- moved J4 0.63 mm to (42.5, 35.6)
- moved R6 0.63 mm to (69.2, 25.4)
Connections:
- removed net N$9: J4.12, S1.2
- new net N$26: J3.2, J6.2
- new net N$34: J4.1, J8.2
- new net N$35: J4.2, J8.3
- new net N$6: J3.3, J6.3
- new net VBAT: C1.1, C2.1, J10.2, J4.12, J9.2, S1.2
- new net VREG: J1.2, J6.4, J8.4, J9.4
- net GND: now also C1.2, C2.2, D1.P$2, J10.1, J6.1, J8.1, J9.3
- net N$17: now also D1.P$1
- net VCC: no longer J1.2
Routing:
- net VREG: track 0.00 -> 140.6 mm
- net VBAT: track 0.00 -> 99.2 mm
- net N$6: track 0.00 -> 66.3 mm
- net N$26: track 0.00 -> 62.7 mm
- net N$35: track 0.00 -> 60.9 mm
- net N$34: track 0.00 -> 56.6 mm
- net VCC: track 95.1 -> 68.7 mm
- net N$9: track 19.4 -> 0.00 mm
- net RST: track 90.2 -> 94.6 mm
- net N$17: track 38.8 -> 39.6 mm
- net N$28: track 66.9 -> 66.2 mm
- net N$29: track 66.9 -> 66.2 mm
- net N$15: track 21.4 -> 20.8 mm
Other:
- board text added: "I2C"
- board text added: "RXD"
- board text added: "SCL"
- board text added: "SDA"
- board text added: "TXD"
- board text added: "UART"
- board text added: "VREG"

Commit message: candidate for final
Parts:
- added J11: (no value), SparkFun-Connectors:1X01
- moved J10 1.27 mm to (73.7, 39.4)
Connections:
- new net N$9: J11.1, J4.9
Routing:
- net N$9: track 0.00 -> 3.17 mm
- net VBAT: track 99.2 -> 97.9 mm
Other:
- board text added: "3.7V Li-Poly 2500mAh Battery"
- board text added: "Adafruit 3.5" 480x320 TFT LCD Breakout Board"
- board text added: "Adafruit Feather FONA 32u4"
- board text added: "Water Level Display V1.0 6/2018"
- board text removed: "Water Level Display V1.0 5/2018"
Changed lines of the file:
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@@
 <text x="9.144" y="19.558" size="1.778" layer="21">Water Level
   Display
-V1.0 5/2018</text>
+V1.0 6/2018</text>
 <wire x1="84.455" y1="36.83" x2="29.21" y2="36.83" width="0" layer="21"/>
 <wire x1="29.21" y1="36.83" x2="26.67" y2="34.29" width="0" layer="21" curve="90"/>
@@
 <hole x="38.1" y="73.66" drill="3.175"/>
 <hole x="38.1" y="58.42" drill="3.175"/>
+<text x="33.274" y="23.368" size="1.778" layer="21">Adafruit Feather
+FONA 32u4</text>
+<text x="53.594" y="47.498" size="1.778" layer="22" rot="MR0">Adafruit 3.5" 480x320
+TFT LCD Breakout Board</text>
+<text x="14.224" y="79.248" size="1.778" layer="21">3.7V Li-Poly 2500mAh Battery</text>
 </plain>
 <attributes>
@@
 <attribute name="PROD_ID" value="CONN-09696" x="67.31" y="8.89" size="1.778" layer="27" rot="R180" display="off"/>
 </element>
-<element name="J10" library="SparkFun-Connectors" package="1X02" value="" x="73.66" y="40.64" smashed="yes">
-<attribute name="NAME" x="71.8312" y="38.6588" size="1.27" layer="25" ratio="10" rot="R90"/>
-<attribute name="VALUE" x="72.39" y="37.465" size="1.27" layer="27"/>
+<element name="J10" library="SparkFun-Connectors" package="1X02" value="" x="73.66" y="39.37" smashed="yes">
+<attribute name="NAME" x="71.8312" y="37.3888" size="1.27" layer="25" ratio="10" rot="R90"/>
+<attribute name="VALUE" x="72.39" y="36.195" size="1.27" layer="27"/>
 </element>
 <element name="C1" library="SparkFun-Capacitors" package="CPOL-RADIAL-100UF-25V" value="330uF" x="77.47" y="29.21" rot="R180"/>
 <element name="C2" library="SparkFun-Capacitors" package="CPOL-RADIAL-100UF-25V" value="330uF" x="77.47" y="21.59" rot="R180"/>
+<element name="J11" library="SparkFun-Connectors" package="1X01" value="" x="62.865" y="38.735"/>
 </elements>
 <signals>
@@
 <contactref element="C1" pad="2"/>
 <contactref element="C2" pad="2"/>
+<via x="45.72" y="7.62" extent="1-16" drill="0.35"/>
 </signal>
 <signal name="VCC">
@@
 <contactref element="S1" pad="2"/>
 <wire x1="86.36" y1="45.72" x2="85.09" y2="45.72" width="1.524" layer="1"/>
-<wire x1="85.09" y1="45.72" x2="78.105" y2="38.735" width="1.524" layer="1"/>
-<wire x1="78.105" y1="38.735" x2="74.295" y2="35.56" width="1.524" layer="1"/>
+<wire x1="85.09" y1="45.72" x2="76.835" y2="38.1" width="1.524" layer="1"/>
+<wire x1="76.835" y1="38.1" x2="74.295" y2="35.56" width="1.524" layer="1"/>
 <wire x1="74.295" y1="35.56" x2="70.485" y2="35.56" width="1.524" layer="1"/>
 <contactref element="J10" pad="2"/>
-<wire x1="76.2" y1="40.64" x2="78.105" y2="38.735" width="1.524" layer="1"/>
+<wire x1="76.2" y1="39.37" x2="76.835" y2="38.1" width="1.524" layer="1"/>
 <contactref element="J9" pad="2"/>
 <wire x1="86.36" y1="45.72" x2="83.82" y2="43.18" width="0.8128" layer="16"/>
@@
 <wire x1="5.08" y1="63.5" x2="2.54" y2="63.5" width="0.8128" layer="1"/>
 </signal>
+<signal name="N$9">
+<contactref element="J4" pad="9"/>
+<contactref element="J11" pad="1"/>
+<wire x1="62.865" y1="38.735" x2="62.865" y2="35.56" width="0.254" layer="16"/>
+</signal>
 </signals>
