File: Eagle/WaterLevelDisplay/WaterLevelDisplay_v1-0.sch (EAGLE design)
At the start: 17 parts, among them J12 POWER_JACKPTH_BREAD, J7 RJ45

Commit message: first round of layout
Parts:
- removed C2: 0.01uF, SparkFun-Passives:CAPPTH1
- removed J10: (no value), SparkFun-Connectors:M02PTH
- removed LED1: (no value), adafruit:LED5MM
- removed R10: 330, resistor:R-US_0204/5
- added CN1: (no value), adafruit:JST_2PIN-SMT-RA
- added J5: (no value), SparkFun-Connectors:M20NOSILK
- added OK1: SFH620A, optocoupler:SFH620A
- R5: value 22K -> 5K
- R6: value 10K -> 8K
Connections:
- removed net MOTION: J7.4
- removed net N$6: C2.1, R5.1, R6.2
- removed net PHOTOCELL: J7.5
- new net CURTRANS_A: J7.4, OK1.AC2
- new net CURTRANS_B: J7.5, OK1.AC1
- new net N$10: J2.8, J5.8
- new net N$11: J2.9, J5.9
- new net N$12: J2.10, J5.10
- new net N$13: J2.11, J5.11
- new net N$14: J2.12, J5.12
- new net N$16: J2.13, J5.13
- new net N$19: J2.14, J5.14
- new net N$2: J2.2, J5.2
- new net N$20: J2.15, J5.15
- new net N$21: J2.16, J5.16
- new net N$22: J2.17, J5.17
- new net N$23: J2.18, J5.18
- new net N$24: J2.19, J5.19
- new net N$25: J2.20, J5.20
- new net N$27: J1.8, J4.7
- new net N$28: J1.19, J3.12
- new net N$29: J1.20, J3.11
- new net N$3: J2.3, J5.3
- new net N$30: J1.10, J4.6
- new net N$31: J3.9, OK1.C
- new net N$32: J1.7, J4.8
- new net N$33: J1.9, J3.7
- new net N$4: J2.4, J5.4
- new net N$5: J2.5, J5.5
- new net N$7: J2.6, J5.6
- new net N$8: J2.7, J5.7
- net GND: now also CN1.1, J1.1, J1.15, J12.GND, J2.1, J3.13, J5.1, OK1.E; no longer C2.2, J10.2, J12.PWR, LED1.C, S11.S
- net MISO: now also J1.5, J3.4
- net MOSI: now also J1.6, J3.5
- net N$1: now also CN1.2, S11.S; no longer LED1.A, R10.2
- net N$15: now also J3.1, J3.8; no longer R10.1
- net N$17: now also J12.PWR, J4.10, R5.2; no longer J10.1, J12.GND
- net N$18: now also J3.10, R5.1, R6.2; no longer R5.2
- net N$9: now also J4.12
- net RST: now also J3.16
- net SCK: now also J1.4, J3.6
- net VCC: now also J1.2, J3.15
Other:
- note added: "1 GND 2 RESET 3 VCC (5V) 4 Current Transformer A 5 Current Transformer B 6 SCK 7 MISO 8 MOSI"
- note added: "3-5V"
- note added: "3.3V out"
- note added: "3V3"
- note added: "AREF"
- note added: "CLK"
- note added: "CS"
- note added: "Card CS"
- note added: "Card Detect"
- note added: "D/C"
- note added: "En"
- note added: "GND"
- note added: "IM0"
- note added: "IM1"
- note added: "IM2"
- note added: "KEY"
- note added: "Lite"
- note added: "MISO"
- note added: "MOSI"
- note added: "PB5"
- note added: "PB6"
- note added: "PB7"
- note added: "PC6"
- note added: "PC7"
- note added: "PD6"
- note added: "PD7"
- note added: "PF0"
- note added: "PF1"
- note added: "PF4"
- note added: "PF5"
- note added: "PF6"
- note added: "PF7"
- note added: "RST"
- note added: "RXD1"
- note added: "SCK"
- note added: "SCL"
- note added: "SDA"
- note added: "TXD1"
- note added: "USB"
- note added: "VBAT"
- note added: "X+"
- note added: "X-"
- note added: "Y+"
- note added: "Y-"
- note removed: "1 GND 2 RESET 3 VCC (5V) 4 motion detector 5 photocell 6 on/off button 7 UART Rx 8 UART Tx"
- note removed: "Battery Charge Input"
- note removed: "LED Indicators"
- moved on the sheet: D11, D7, D8, D9, J12, J2, J3, J4, J7, R5, R6, S11

Commit message: Add files via upload
Parts:
- added C1, C2: 330uF, SparkFun-Capacitors:CAP_POLPTH1
- added D1: 6V Zener, SparkFun-DiscreteSemi:DIODE-ZENERPTH
- added J10: (no value), SparkFun-Connectors:M02PTH
- added J6, J8, J9: (no value), SparkFun-Connectors:M04PTH
Connections:
- removed net N$9: J4.12, S11.P
- new net N$26: J3.2, J6.2
- new net N$34: J4.1, J8.2
- new net N$35: J4.2, J8.3
- new net N$6: J3.3, J6.3
- new net VBAT: C1.+, C2.+, J10.2, J4.12, J9.2, S11.P
- new net VREG: J1.2, J6.4, J8.4, J9.4
- net GND: now also C1.-, C2.-, D1.A, J10.1, J6.1, J8.1, J9.3
- net N$17: now also D1.C
- net VCC: no longer J1.2
Other:
- note added: "Adafruit 3.5" TFT Display Module"
- note added: "Adafruit Feather FONA"
- note added: "I2C"
- note added: "Pololu S7V8F3"
- note added: "SHDN"
- note added: "VIN"
- note added: "VOUT"
- note added: "VREG"
- moved on the sheet: CN1, J12, J3, J4, R5, R6, S11

Commit message: candidate for final
Parts:
- added J11: (no value), SparkFun-Connectors:M01PTH
Connections:
- new net N$9: J11.1, J4.9
Other:
- note added: "Mains Detection"
- note added: "Pump On Detection"
- moved on the sheet: D1
Changed lines of the file:
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@@
 <part name="GND13" library="SparkFun-Aesthetics" deviceset="GND" device=""/>
 <part name="GND14" library="SparkFun-Aesthetics" deviceset="GND" device=""/>
+<part name="J11" library="SparkFun-Connectors" deviceset="M01" device="PTH"/>
 </parts>
 <sheets>
 <sheet>
 <plain>
-<text x="-76.2" y="152.4" size="1.778" layer="97" align="bottom-right">Mains
-Detector</text>
+<text x="45.212" y="183.896" size="1.778" layer="97" align="bottom-right">Mains
+Detection</text>
 <text x="-64.77" y="95.25" size="1.6764" layer="91" align="top-left">1 GND
 2 RESET
@@
 <text x="87.884" y="146.812" size="1.778" layer="91">SDA</text>
 <text x="87.884" y="144.272" size="1.778" layer="91">GND</text>
+<text x="-76.708" y="153.416" size="1.778" layer="97" align="bottom-right">Pump On
+Detection</text>
 </plain>
 <instances>
@@
 <instance part="CN1" gate="G$1" x="132.08" y="195.58"/>
 <instance part="GND6" gate="1" x="121.92" y="190.5"/>
-<instance part="D1" gate="G$1" x="116.84" y="152.4" rot="R90"/>
-<instance part="GND8" gate="1" x="116.84" y="142.24"/>
+<instance part="D1" gate="G$1" x="119.38" y="152.4" rot="R90"/>
+<instance part="GND8" gate="1" x="119.38" y="142.24"/>
 <instance part="J6" gate="G$1" x="-27.94" y="144.78"/>
 <instance part="J8" gate="G$1" x="81.28" y="147.32" rot="MR0"/>
@@
 <instance part="GND13" gate="1" x="78.74" y="177.8"/>
 <instance part="GND14" gate="1" x="66.04" y="177.8"/>
+<instance part="J11" gate="G$1" x="78.74" y="165.1" rot="R180"/>
 </instances>
 <busses>
@@
 <pinref part="D1" gate="G$1" pin="A"/>
 <pinref part="GND8" gate="1" pin="GND"/>
-<wire x1="116.84" y1="149.86" x2="116.84" y2="144.78" width="0.1524" layer="91"/>
+<wire x1="119.38" y1="149.86" x2="119.38" y2="144.78" width="0.1524" layer="91"/>
 </segment>
 <segment>
@@
 <pinref part="J12" gate="G$1" pin="PWR"/>
 <wire x1="121.92" y1="177.8" x2="119.38" y2="177.8" width="0.1524" layer="91"/>
-<wire x1="119.38" y1="177.8" x2="116.84" y2="165.1" width="0.1524" layer="91"/>
-<wire x1="116.84" y1="165.1" x2="88.9" y2="165.1" width="0.1524" layer="91"/>
+<wire x1="119.38" y1="177.8" x2="119.38" y2="165.1" width="0.1524" layer="91"/>
+<wire x1="119.38" y1="165.1" x2="88.9" y2="165.1" width="0.1524" layer="91"/>
 <wire x1="88.9" y1="165.1" x2="88.9" y2="170.18" width="0.1524" layer="91"/>
 <wire x1="88.9" y1="170.18" x2="58.42" y2="170.18" width="0.1524" layer="91"/>
 <junction x="58.42" y="170.18"/>
 <pinref part="D1" gate="G$1" pin="C"/>
-<wire x1="116.84" y1="154.94" x2="116.84" y2="165.1" width="0.1524" layer="91"/>
-<junction x="116.84" y="165.1"/>
+<wire x1="119.38" y1="154.94" x2="119.38" y2="165.1" width="0.1524" layer="91"/>
+<junction x="119.38" y="165.1"/>
 </segment>
 </net>
@@
 </segment>
 </net>
+<net name="N$9" class="0">
+<segment>
+<pinref part="J4" gate="G$1" pin="9"/>
+<wire x1="55.88" y1="167.64" x2="68.58" y2="167.64" width="0.1524" layer="91"/>
+<wire x1="68.58" y1="167.64" x2="68.58" y2="165.1" width="0.1524" layer="91"/>
+<pinref part="J11" gate="G$1" pin="1"/>
+<wire x1="68.58" y1="165.1" x2="71.12" y2="165.1" width="0.1524" layer="91"/>
+</segment>
+</net>
